File: hardware/RAPTOR/RAPTOR.sch (KiCad schematic (older format))
At the start: 13 parts, among them P1 Digital, P10 CONN_01X01, P11 CONN_01X01, P12 CONN_01X01, P13 CONN_01X01, P2 Power, P3 Analog, P4 Analog, P5 PWM, P6 PWM, P7 Communication, P8 CONN_01X01, P9 CONN_01X01

Commit message: add BMP280 and wiring
Parts:
- added U?: BMP280, LGA-8-2.5X2.5, symbol SparkFun-Sensors:BMP280
Connections:
- wire segments 96 -> 105
Changed lines of the file:
@@
 EESchema Schematic File Version 4
-LIBS:Arduino_Mega-cache
+LIBS:RAPTOR-cache
 EELAYER 26 0
 EELAYER END
@@
 Wire Notes Line
 	8350 6050 8350 500
+$Comp
+L SparkFun-Sensors:BMP280 U?
+U 1 1 5BD37EBF
+P 2250 1800
+F 0 "U?" H 2250 2360 45  0000 C CNN
+F 1 "BMP280" H 2250 2276 45  0000 C CNN
+F 2 "LGA-8-2.5X2.5" H 2250 2250 20  0001 C CNN
+F 3 "" H 2250 1800 60  0001 C CNN
+F 4 "IC-13090" H 2250 2181 60  0000 C CNN "Field4"
+	1    2250 1800
+	1    0    0    -1
+$EndComp
+Wire Wire Line
+	1700 1800 1650 1800
+Wire Wire Line
+	1650 1800 1650 1600
+Wire Wire Line
+	1650 1600 1700 1600
+Wire Wire Line
+	1650 1600 1550 1600
+Wire Wire Line
+	1550 1600 1550 1500
+Connection ~ 1650 1600
+$Comp
+L power:GND #PWR?
+U 1 1 5BD3E0CC
+P 1550 2150
+F 0 "#PWR?" H 1550 1900 50  0001 C CNN
+F 1 "GND" H 1555 1977 50  0000 C CNN
+F 2 "" H 1550 2150 50  0001 C CNN
+F 3 "" H 1550 2150 50  0001 C CNN
+	1    1550 2150
+	1    0    0    -1
+$EndComp
+Wire Wire Line
+	1700 2100 1550 2100
+Wire Wire Line
+	1550 2100 1550 2150
+$Comp
+L power:+5V #PWR?
+U 1 1 5BD412DA
+P 1550 1500
+F 0 "#PWR?" H 1550 1350 50  0001 C CNN
+F 1 "+5V" H 1565 1673 50  0000 C CNN
+F 2 "" H 1550 1500 50  0001 C CNN
+F 3 "" H 1550 1500 50  0001 C CNN
+	1    1550 1500
+	1    0    0    -1
+$EndComp
+Text Label 3050 1900 0    50   ~ 0
+21(SCL)
+Wire Wire Line
+	2800 1900 3050 1900
+Text Label 3050 1800 0    50   ~ 0
+20(SDA)
+Wire Wire Line
+	2800 1800 3050 1800
 $EndSCHEMATC

Commit message: make pcb
Parts:
- gave numbers to parts that had none: 1
Changed lines of the file:
@@
 	8350 6050 8350 500
 $Comp
-L SparkFun-Sensors:BMP280 U?
+L SparkFun-Sensors:BMP280 U1
 U 1 1 5BD37EBF
 P 2250 1800
-F 0 "U?" H 2250 2360 45  0000 C CNN
+F 0 "U1" H 2250 2360 45  0000 C CNN
 F 1 "BMP280" H 2250 2276 45  0000 C CNN
 F 2 "LGA-8-2.5X2.5" H 2250 2250 20  0001 C CNN
@@
 Connection ~ 1650 1600
 $Comp
-L power:GND #PWR?
+L power:GND #PWR0101
 U 1 1 5BD3E0CC
 P 1550 2150
-F 0 "#PWR?" H 1550 1900 50  0001 C CNN
+F 0 "#PWR0101" H 1550 1900 50  0001 C CNN
 F 1 "GND" H 1555 1977 50  0000 C CNN
 F 2 "" H 1550 2150 50  0001 C CNN
@@
 	1550 2100 1550 2150
 $Comp
-L power:+5V #PWR?
+L power:+5V #PWR0102
 U 1 1 5BD412DA
 P 1550 1500
-F 0 "#PWR?" H 1550 1350 50  0001 C CNN
+F 0 "#PWR0102" H 1550 1350 50  0001 C CNN
 F 1 "+5V" H 1565 1673 50  0000 C CNN
 F 2 "" H 1550 1500 50  0001 C CNN

Commit message: add bmp footprint
Parts:
- U1: footprint LGA-8-2.5X2.5 -> Silicon-Standard:LGA-8-2.5X2.5
Changed lines of the file:
@@
 F 0 "U1" H 2250 2360 45  0000 C CNN
 F 1 "BMP280" H 2250 2276 45  0000 C CNN
-F 2 "LGA-8-2.5X2.5" H 2250 2250 20  0001 C CNN
+F 2 "Silicon-Standard:LGA-8-2.5X2.5" H 2250 2250 20  0001 C CNN
 F 3 "" H 2250 1800 60  0001 C CNN
 F 4 "IC-13090" H 2250 2181 60  0000 C CNN "Field4"

Commit message: move to uno, re-add bmp
Parts:
- removed P1: Digital, Socket_Arduino_Mega:Socket_Strip_Arduino_2x18, symbol Connector_Generic:Conn_02x18_Odd_Even
- removed P10, P11, P12, P13, P9: CONN_01X01, Socket_Arduino_Mega:Arduino_1pin, symbol Connector_Generic:Conn_01x01
- removed P2: Power, Socket_Arduino_Mega:Socket_Strip_Arduino_1x08, symbol Connector_Generic:Conn_01x08
- removed P3: Analog, Socket_Arduino_Mega:Socket_Strip_Arduino_1x08, symbol Connector_Generic:Conn_01x08
- removed P5: PWM, Socket_Arduino_Mega:Socket_Strip_Arduino_1x10, symbol Connector_Generic:Conn_01x10
- removed P6: PWM, Socket_Arduino_Mega:Socket_Strip_Arduino_1x08, symbol Connector_Generic:Conn_01x08
- removed P7: Communication, Socket_Arduino_Mega:Socket_Strip_Arduino_1x08, symbol Connector_Generic:Conn_01x08
- removed U1: BMP280, Silicon-Standard:LGA-8-2.5X2.5, symbol SparkFun-Sensors:BMP280
- added P1: Power, Socket_Arduino_Uno:Socket_Strip_Arduino_1x08, symbol Connector_Generic:Conn_01x08
- added P2: Analog, Socket_Arduino_Uno:Socket_Strip_Arduino_1x06, symbol Connector_Generic:Conn_01x06
- added P3: Digital, Socket_Arduino_Uno:Socket_Strip_Arduino_1x10, symbol Connector_Generic:Conn_01x10
- added P5, P6, P7: CONN_01X01, Socket_Arduino_Uno:Arduino_1pin, symbol Connector_Generic:Conn_01x01
- P4: value Analog -> Digital; footprint Socket_Arduino_Mega:Socket_Strip_Arduino_1x08 -> Socket_Arduino_Uno:Socket_Strip_Arduino_1x08
- P8: footprint Socket_Arduino_Mega:Arduino_1pin -> Socket_Arduino_Uno:Arduino_1pin
Connections:
- net labels added: 0(Rx), 1(Tx), 10(**/SS), 11(**/MOSI), 12(MISO), 13(SCK), 2, 4, 7, 8, A4(SDA), A5(SCL)
- net labels removed: 0(Rx0), 1(Tx0), 10(**), 11(**), 12(**), 13(**), 14(Tx3), 15(Rx3), 16(Tx2), 17(Rx2), 18(Tx1), 19(Rx1), 2(**), 20(SDA), 21(SCL), 22, 23, 24, 25, 26, 27, 28, 29, 30, 31, 32, 33, 34, 35, 36, 37, 38, 39, 4(**), 40, 41, 42, 43, 44, 45, 46, 47, 48, 49, 50(MISO), 51(MOSI), 52(SCK), 53(SS), 7(**), 8(**), A10, A11, A12, A13, A14, A15, A4, A5, A6, A7, A8, A9, SCL, SDA
- wire segments 105 -> 38
- no-connect marks 7 -> 5
Other:
- note added: "Shield for Arduino that uses\nthe same pin disposition\nlike "Uno" board Rev 3."
- note removed: "Shield for Arduino Mega Rev 3"

Commit message: add bno, start on footprint for bmp
Parts:
- added U1: BMP280, Silicon-Standard:LGA-8-2.5X2.5, symbol SparkFun-Sensors:BMP280
- added U2: BNO055, Silicon-Standard:LGA-8-2.5X2.5, symbol SparkFun-Sensors:BNO055
Connections:
- wire segments 38 -> 50
Changed lines of the file:
@@
 EESchema Schematic File Version 4
-LIBS:Arduino_As_Uno-cache
+LIBS:RAPTOR-cache
 EELAYER 26 0
 EELAYER END
@@
 Wire Notes Line
 	10700 1000 10700 500
+$Comp
+L SparkFun-Sensors:BMP280 U1
+U 1 1 5BD31CAC
+P 2300 1700
+F 0 "U1" H 2300 2154 45  0000 C CNN
+F 1 "BMP280" H 2300 2070 45  0000 C CNN
+F 2 "Silicon-Standard:LGA-8-2.5X2.5" H 2300 2150 20  0001 C CNN
+F 3 "" H 2300 1700 60  0001 C CNN
+	1    2300 1700
+	1    0    0    -1
+$EndComp
+$Comp
+L power:+5V #PWR0101
+U 1 1 5BD35138
+P 1550 1400
+F 0 "#PWR0101" H 1550 1250 50  0001 C CNN
+F 1 "+5V" H 1565 1573 50  0000 C CNN
+F 2 "" H 1550 1400 50  0001 C CNN
+F 3 "" H 1550 1400 50  0001 C CNN
+	1    1550 1400
+	1    0    0    -1
+$EndComp
+Wire Wire Line
+	1550 1400 1550 1500
+Wire Wire Line
+	1550 1500 1750 1500
+$Comp
+L power:GND #PWR0102
+U 1 1 5BD35A48
+P 1550 2100
+F 0 "#PWR0102" H 1550 1850 50  0001 C CNN
+F 1 "GND" H 1555 1927 50  0000 C CNN
+F 2 "" H 1550 2100 50  0001 C CNN
+F 3 "" H 1550 2100 50  0001 C CNN
+	1    1550 2100
+	1    0    0    -1
+$EndComp
+Wire Wire Line
+	1750 2000 1550 2000
+Wire Wire Line
+	1550 2000 1550 2100
+Text Label 3200 1800 0    50   ~ 0
+A5(SCL)
+Text Label 3200 1700 0    50   ~ 0
+A4(SDA)
+Wire Wire Line
+	2850 1700 3200 1700
+Wire Wire Line
+	2850 1800 3200 1800
+$Comp
+L SparkFun-Sensors:BNO055 U2
+U 1 1 5BD45163
+P 2300 4050
+F 0 "U2" H 2300 4504 45  0000 C CNN
+F 1 "BNO055" H 2300 4420 45  0000 C CNN
+F 2 "Silicon-Standard:LGA-8-2.5X2.5" H 2300 4500 20  0001 C CNN
+F 3 "" H 2300 4050 60  0001 C CNN
+	1    2300 4050
+	1    0    0    -1
+$EndComp
+$Comp
+L power:+5V #PWR0103
+U 1 1 5BD4727B
+P 1550 3750
+F 0 "#PWR0103" H 1550 3600 50  0001 C CNN
+F 1 "+5V" H 1565 3923 50  0000 C CNN
+F 2 "" H 1550 3750 50  0001 C CNN
+F 3 "" H 1550 3750 50  0001 C CNN
+	1    1550 3750
+	1    0    0    -1
+$EndComp
+Wire Wire Line
+	1550 3750 1550 3850
+Wire Wire Line
+	1550 3850 1750 3850
+$Comp
+L power:GND #PWR0104
+U 1 1 5BD47283
+P 1550 4450
+F 0 "#PWR0104" H 1550 4200 50  0001 C CNN
+F 1 "GND" H 1555 4277 50  0000 C CNN
+F 2 "" H 1550 4450 50  0001 C CNN
+F 3 "" H 1550 4450 50  0001 C CNN
+	1    1550 4450
+	1    0    0    -1
+$EndComp
+Wire Wire Line
+	1750 4350 1550 4350
+Wire Wire Line
+	1550 4350 1550 4450
+Text Label 3200 4050 0    50   ~ 0
+A5(SCL)
+Text Label 3200 3900 0    50   ~ 0
+A4(SDA)
+Wire Wire Line
+	2850 4050 3200 4050
+Wire Wire Line
+	2850 3900 3200 3900
 $EndSCHEMATC
