File: hardware/RAPTOR/RAPTOR.sch (KiCad schematic (older format))
At the start: 10 parts, among them P1 Power, P2 Analog, P3 Digital, P4 Digital, P5 CONN_01X01, P6 CONN_01X01, P7 CONN_01X01, P8 CONN_01X01, U1 BMP280, U2 BNO055

Commit message: small changes to gps symbol, add gps and openlog to schematic
Parts:
- added U?: AdafruitGPS, symbol adafruitgps:AdafruitGPS
- added U?: OpenLog, LGA-8-2.5X2.5, symbol openlog:OpenLog
- U1: symbol SparkFun-Sensors:BMP280 -> bmp280:BMP280
- U2: symbol SparkFun-Sensors:BNO055 -> bno055:BNO055
Connections:
- net labels added: FIX_LED
- wire segments 50 -> 63
- no-connect marks 5 -> 15
Changed lines of the file:
@@
 encoding utf-8
 Sheet 1 1
-Title ""
-Date "lun. 30 mars 2015"
-Rev ""
+Title "RAPTOR Schematic"
+Date "2018-11-03"
+Rev "FALCON"
 Comp ""
 Comment1 ""
@@
 	10700 1000 10700 500
 $Comp
-L SparkFun-Sensors:BMP280 U1
+L bmp280:BMP280 U1
 U 1 1 5BD31CAC
 P 2300 1700
@@
 	2850 1800 3200 1800
 $Comp
-L SparkFun-Sensors:BNO055 U2
+L bno055:BNO055 U2
 U 1 1 5BD45163
-P 2300 4050
-F 0 "U2" H 2300 4504 45  0000 C CNN
-F 1 "BNO055" H 2300 4420 45  0000 C CNN
-F 2 "Silicon-Standard:LGA-8-2.5X2.5" H 2300 4500 20  0001 C CNN
-F 3 "" H 2300 4050 60  0001 C CNN
-	1    2300 4050
+P 2300 3200
+F 0 "U2" H 2300 3654 45  0000 C CNN
+F 1 "BNO055" H 2300 3570 45  0000 C CNN
+F 2 "Silicon-Standard:LGA-8-2.5X2.5" H 2300 3650 20  0001 C CNN
+F 3 "" H 2300 3200 60  0001 C CNN
+	1    2300 3200
 	1    0    0    -1
 $EndComp
@@
 L power:+5V #PWR0103
 U 1 1 5BD4727B
-P 1550 3750
-F 0 "#PWR0103" H 1550 3600 50  0001 C CNN
-F 1 "+5V" H 1565 3923 50  0000 C CNN
-F 2 "" H 1550 3750 50  0001 C CNN
-F 3 "" H 1550 3750 50  0001 C CNN
-	1    1550 3750
-	1    0    0    -1
-$EndComp
-Wire Wire Line
-	1550 3750 1550 3850
-Wire Wire Line
-	1550 3850 1750 3850
+P 1550 2900
+F 0 "#PWR0103" H 1550 2750 50  0001 C CNN
+F 1 "+5V" H 1565 3073 50  0000 C CNN
+F 2 "" H 1550 2900 50  0001 C CNN
+F 3 "" H 1550 2900 50  0001 C CNN
+	1    1550 2900
+	1    0    0    -1
+$EndComp
+Wire Wire Line
+	1550 2900 1550 3000
+Wire Wire Line
+	1550 3000 1750 3000
 $Comp
 L power:GND #PWR0104
 U 1 1 5BD47283
-P 1550 4450
-F 0 "#PWR0104" H 1550 4200 50  0001 C CNN
-F 1 "GND" H 1555 4277 50  0000 C CNN
-F 2 "" H 1550 4450 50  0001 C CNN
-F 3 "" H 1550 4450 50  0001 C CNN
-	1    1550 4450
-	1    0    0    -1
-$EndComp
-Wire Wire Line
-	1750 4350 1550 4350
-Wire Wire Line
-	1550 4350 1550 4450
-Text Label 3200 4050 0    50   ~ 0
+P 1550 3600
+F 0 "#PWR0104" H 1550 3350 50  0001 C CNN
+F 1 "GND" H 1555 3427 50  0000 C CNN
+F 2 "" H 1550 3600 50  0001 C CNN
+F 3 "" H 1550 3600 50  0001 C CNN
+	1    1550 3600
+	1    0    0    -1
+$EndComp
+Wire Wire Line
+	1750 3500 1550 3500
+Wire Wire Line
+	1550 3500 1550 3600
+Text Label 3200 3200 0    50   ~ 0
 A5(SCL)
-Text Label 3200 3900 0    50   ~ 0
+Text Label 3200 3050 0    50   ~ 0
 A4(SDA)
 Wire Wire Line
-	2850 4050 3200 4050
-Wire Wire Line
-	2850 3900 3200 3900
+	2850 3200 3200 3200
+Wire Wire Line
+	2850 3050 3200 3050
+$Comp
+L openlog:OpenLog U?
+U 1 1 5BDE8282
+P 2300 4500
+F 0 "U?" H 2300 4954 45  0000 C CNN
+F 1 "OpenLog" H 2300 4870 45  0000 C CNN
+F 2 "LGA-8-2.5X2.5" H 2300 4950 20  0001 C CNN
+F 3 "" H 2300 4500 60  0001 C CNN
+	1    2300 4500
+	1    0    0    -1
+$EndComp
+$Comp
+L adafruitgps:AdafruitGPS U?
+U 1 1 5BDE25E6
+P 2450 5950
+F 0 "U?" H 2450 6475 50  0000 C CNN
+F 1 "AdafruitGPS" H 2450 6384 50  0000 C CNN
+F 2 "" H 2550 5900 50  0001 C CNN
+F 3 "" H 2550 5900 50  0001 C CNN
+	1    2450 5950
+	1    0    0    -1
+$EndComp
+Text Label 3200 4750 0    50   ~ 0
+0(Rx)
+Wire Wire Line
+	2850 4750 3200 4750
+Text Label 3200 4350 0    50   ~ 0
+1(Tx)
+Wire Wire Line
+	2850 4350 3200 4350
+$Comp
+L power:GND #PWR?
+U 1 1 5BDE53C7
+P 1550 4900
+F 0 "#PWR?" H 1550 4650 50  0001 C CNN
+F 1 "GND" H 1555 4727 50  0000 C CNN
+F 2 "" H 1550 4900 50  0001 C CNN
+F 3 "" H 1550 4900 50  0001 C CNN
+	1    1550 4900
+	1    0    0    -1
+$EndComp
+Wire Wire Line
+	1750 4800 1550 4800
+Wire Wire Line
+	1550 4800 1550 4900
+$Comp
+L power:GND #PWR?
+U 1 1 5BDE7CE6
+P 1550 6400
+F 0 "#PWR?" H 1550 6150 50  0001 C CNN
+F 1 "GND" H 1555 6227 50  0000 C CNN
+F 2 "" H 1550 6400 50  0001 C CNN
+F 3 "" H 1550 6400 50  0001 C CNN
+	1    1550 6400
+	1    0    0    -1
+$EndComp
+Wire Wire Line
+	1750 6300 1550 6300
+Wire Wire Line
+	1550 6300 1550 6400
+$Comp
+L power:+5V #PWR?
+U 1 1 5BDE90FA
+P 1550 5600
+F 0 "#PWR?" H 1550 5450 50  0001 C CNN
+F 1 "+5V" H 1565 5773 50  0000 C CNN
+F 2 "" H 1550 5600 50  0001 C CNN
+F 3 "" H 1550 5600 50  0001 C CNN
+	1    1550 5600
+	1    0    0    -1
+$EndComp
+Wire Wire Line
+	1550 5600 1550 5700
+Wire Wire Line
+	1550 5700 1750 5700
+$Comp
+L power:+5V #PWR?
+U 1 1 5BDEA4F5
+P 1550 4250
+F 0 "#PWR?" H 1550 4100 50  0001 C CNN
+F 1 "+5V" H 1565 4423 50  0000 C CNN
+F 2 "" H 1550 4250 50  0001 C CNN
+F 3 "" H 1550 4250 50  0001 C CNN
+	1    1550 4250
+	1    0    0    -1
+$EndComp
+Wire Wire Line
+	1550 4250 1550 4350
+Wire Wire Line
+	1550 4350 1750 4350
+Text Label 3500 5800 0    50   ~ 0
+3(**)
+Wire Wire Line
+	3150 5800 3500 5800
+Text Label 3500 5950 0    50   ~ 0
+2
+Wire Wire Line
+	3150 5950 3500 5950
+Text Label 3500 6250 0    50   ~ 0
+FIX_LED
+Wire Wire Line
+	3150 6250 3500 6250
+NoConn ~ 1750 5800
+NoConn ~ 1750 5950
+NoConn ~ 3150 6100
+NoConn ~ 3150 5650
+NoConn ~ 1750 4600
+NoConn ~ 1750 4700
+NoConn ~ 1750 3200
+NoConn ~ 1750 1700
+NoConn ~ 2850 1500
+NoConn ~ 2850 2000
 $EndSCHEMATC

Commit message: Added all the footprints and associated them with the symbols in the schematics
Parts:
- U1: footprint Silicon-Standard:LGA-8-2.5X2.5 -> RAPTOR_footprints:BMP280; symbol bmp280:BMP280 -> RAPTOR-rescue:BMP280-bmp280
- U2: footprint Silicon-Standard:LGA-8-2.5X2.5 -> RAPTOR_footprints:BNO055; symbol bno055:BNO055 -> RAPTOR-rescue:BNO055-bno055
- U3: renamed from U?; footprint LGA-8-2.5X2.5 -> RAPTOR_footprints:OpenLog; symbol openlog:OpenLog -> RAPTOR-rescue:OpenLog-openlog
- U4: renamed from U?; footprint (none) -> RAPTOR_footprints:AdafruitGPS; symbol adafruitgps:AdafruitGPS -> RAPTOR-rescue:AdafruitGPS-adafruitgps
Changed lines of the file:
@@
 	10700 1000 10700 500
 $Comp
-L bmp280:BMP280 U1
+L RAPTOR-rescue:BMP280-bmp280 U1
 U 1 1 5BD31CAC
 P 2300 1700
 F 0 "U1" H 2300 2154 45  0000 C CNN
 F 1 "BMP280" H 2300 2070 45  0000 C CNN
-F 2 "Silicon-Standard:LGA-8-2.5X2.5" H 2300 2150 20  0001 C CNN
+F 2 "RAPTOR_footprints:BMP280" H 2300 2150 20  0001 C CNN
 F 3 "" H 2300 1700 60  0001 C CNN
 	1    2300 1700
@@
 	2850 1800 3200 1800
 $Comp
-L bno055:BNO055 U2
+L RAPTOR-rescue:BNO055-bno055 U2
 U 1 1 5BD45163
 P 2300 3200
 F 0 "U2" H 2300 3654 45  0000 C CNN
 F 1 "BNO055" H 2300 3570 45  0000 C CNN
-F 2 "Silicon-Standard:LGA-8-2.5X2.5" H 2300 3650 20  0001 C CNN
+F 2 "RAPTOR_footprints:BNO055" H 2300 3650 20  0001 C CNN
 F 3 "" H 2300 3200 60  0001 C CNN
 	1    2300 3200
@@
 	2850 3050 3200 3050
 $Comp
-L openlog:OpenLog U?
+L RAPTOR-rescue:OpenLog-openlog U3
 U 1 1 5BDE8282
 P 2300 4500
-F 0 "U?" H 2300 4954 45  0000 C CNN
+F 0 "U3" H 2300 4954 45  0000 C CNN
 F 1 "OpenLog" H 2300 4870 45  0000 C CNN
-F 2 "LGA-8-2.5X2.5" H 2300 4950 20  0001 C CNN
+F 2 "RAPTOR_footprints:OpenLog" H 2300 4950 20  0001 C CNN
 F 3 "" H 2300 4500 60  0001 C CNN
 	1    2300 4500
@@
 $EndComp
 $Comp
-L adafruitgps:AdafruitGPS U?
+L RAPTOR-rescue:AdafruitGPS-adafruitgps U4
 U 1 1 5BDE25E6
 P 2450 5950
-F 0 "U?" H 2450 6475 50  0000 C CNN
+F 0 "U4" H 2450 6475 50  0000 C CNN
 F 1 "AdafruitGPS" H 2450 6384 50  0000 C CNN
-F 2 "" H 2550 5900 50  0001 C CNN
+F 2 "RAPTOR_footprints:AdafruitGPS" H 2550 5900 50  0001 C CNN
 F 3 "" H 2550 5900 50  0001 C CNN
 	1    2450 5950
@@
 	2850 4350 3200 4350
 $Comp
-L power:GND #PWR?
+L power:GND #PWR0105
 U 1 1 5BDE53C7
 P 1550 4900
-F 0 "#PWR?" H 1550 4650 50  0001 C CNN
+F 0 "#PWR0105" H 1550 4650 50  0001 C CNN
 F 1 "GND" H 1555 4727 50  0000 C CNN
 F 2 "" H 1550 4900 50  0001 C CNN
@@
 	1550 4800 1550 4900
 $Comp
-L power:GND #PWR?
+L power:GND #PWR0106
 U 1 1 5BDE7CE6
 P 1550 6400
-F 0 "#PWR?" H 1550 6150 50  0001 C CNN
+F 0 "#PWR0106" H 1550 6150 50  0001 C CNN
 F 1 "GND" H 1555 6227 50  0000 C CNN
 F 2 "" H 1550 6400 50  0001 C CNN
@@
 	1550 6300 1550 6400
 $Comp
-L power:+5V #PWR?
+L power:+5V #PWR0107
 U 1 1 5BDE90FA
 P 1550 5600
-F 0 "#PWR?" H 1550 5450 50  0001 C CNN
+F 0 "#PWR0107" H 1550 5450 50  0001 C CNN
 F 1 "+5V" H 1565 5773 50  0000 C CNN
 F 2 "" H 1550 5600 50  0001 C CNN
@@
 	1550 5700 1750 5700
 $Comp
-L power:+5V #PWR?
+L power:+5V #PWR0108
 U 1 1 5BDEA4F5
 P 1550 4250
-F 0 "#PWR?" H 1550 4100 50  0001 C CNN
+F 0 "#PWR0108" H 1550 4100 50  0001 C CNN
 F 1 "+5V" H 1565 4423 50  0000 C CNN
 F 2 "" H 1550 4250 50  0001 C CNN

Commit message: fix sensor numbers, add servos, solenoids, leds, switches
Parts:
- added BZ?: Buzzer, symbol Device:Buzzer
- added D?: LED, symbol Device:LED
- added D? (x3): SOLP_LED, symbol Device:LED
- added D? (x3): SOLC_LED, symbol Device:LED
- added M? (x2): Motor_Servo, symbol Motor:Motor_Servo
- added Q? (x4): MOSFET-NCH-2N7002PW, SOT323, symbol SparkFun-DiscreteSemi:MOSFET-NCH-2N7002PW
- added SOLC, SOLP: -12V, symbol power:-12V
- added SW?: EEPROM_BTN, symbol Switch:SW_SPST
- added SW?: SOLP_SW, symbol Switch:SW_SPST
- added SW?: SOLC_SW, symbol Switch:SW_SPST
Connections:
- net labels added: +12V, +6V, 11, 12
- wire segments 63 -> 117

Commit message: add net + pcb files
Parts:
- removed SOLC, SOLP: -12V, symbol power:-12V
- gave numbers to parts that had none: 17
Connections:
- net labels added: -12V
Changed lines of the file:
@@
 NoConn ~ 2850 2000
 $Comp
-L Motor:Motor_Servo M?
+L Motor:Motor_Servo M1
 U 1 1 5BE79CAA
 P 4300 1700
-F 0 "M?" H 4296 1393 50  0000 C CNN
+F 0 "M1" H 4296 1393 50  0000 C CNN
 F 1 "Motor_Servo" H 4296 1484 50  0000 C CNN
 F 2 "" H 4300 1510 50  0001 C CNN
@@
 	4600 1800 5000 1800
 $Comp
-L power:+6V #PWR?
+L power:+6V #PWR0109
 U 1 1 5BE7EDED
 P 4900 1550
-F 0 "#PWR?" H 4900 1400 50  0001 C CNN
+F 0 "#PWR0109" H 4900 1400 50  0001 C CNN
 F 1 "+6V" H 4915 1723 50  0000 C CNN
 F 2 "" H 4900 1550 50  0001 C CNN
@@
 $EndComp
 $Comp
-L power:GND #PWR?
+L power:GND #PWR0110
 U 1 1 5BE823AD
 P 4750 1400
-F 0 "#PWR?" H 4750 1150 50  0001 C CNN
+F 0 "#PWR0110" H 4750 1150 50  0001 C CNN
 F 1 "GND" H 4755 1227 50  0000 C CNN
 F 2 "" H 4750 1400 50  0001 C CNN
@@
 	4900 1700 4900 1550
 $Comp
-L Motor:Motor_Servo M?
+L Motor:Motor_Servo M2
 U 1 1 5BE85BA8
 P 4300 2500
-F 0 "M?" H 4296 2193 50  0000 C CNN
+F 0 "M2" H 4296 2193 50  0000 C CNN
 F 1 "Motor_Servo" H 4296 2284 50  0000 C CNN
 F 2 "" H 4300 2310 50  0001 C CNN
@@
 	4600 2600 5000 2600
 $Comp
-L power:+6V #PWR?
+L power:+6V #PWR0111
 U 1 1 5BE85BB1
 P 4900 2350
-F 0 "#PWR?" H 4900 2200 50  0001 C CNN
+F 0 "#PWR0111" H 4900 2200 50  0001 C CNN
 F 1 "+6V" H 4915 2523 50  0000 C CNN
 F 2 "" H 4900 2350 50  0001 C CNN
@@
 $EndComp
 $Comp
-L power:GND #PWR?
+L power:GND #PWR0112
 U 1 1 5BE85BB7
 P 4750 2200
-F 0 "#PWR?" H 4750 1950 50  0001 C CNN
+F 0 "#PWR0112" H 4750 1950 50  0001 C CNN
 F 1 "GND" H 4755 2027 50  0000 C CNN
 F 2 "" H 4750 2200 50  0001 C CNN
@@
 	4900 2500 4900 2350
 $Comp
-L power:-12V SOLP
+L power:-12V #SOLP0101
 U 1 1 5BE89FE1
 P 4650 3600
-F 0 "SOLP" H 4592 3591 50  0000 R CNN
+F 0 "#SOLP0101" H 4592 3591 50  0000 R CNN
 F 1 "-12V" H 4592 3682 50  0000 R CNN
 F 2 "" H 4650 3600 50  0001 C CNN
@@
 $EndComp
 $Comp
-L power:+12V #PWR?
+L power:+12V #PWR0113
 U 1 1 5BE8A086
 P 4650 3000
-F 0 "#PWR?" H 4650 2850 50  0001 C CNN
+F 0 "#PWR0113" H 4650 2850 50  0001 C CNN
 F 1 "+12V" H 4665 3173 50  0000 C CNN
 F 2 "" H 4650 3000 50  0001 C CNN
@@
 $EndComp
 $Comp
-L SparkFun-DiscreteSemi:MOSFET-NCH-2N7002PW Q?
+L SparkFun-DiscreteSemi:MOSFET-NCH-2N7002PW Q1
 U 1 1 5BE8A581
 P 4550 3300
-F 0 "Q?" H 4715 3395 45  0000 L CNN
+F 0 "Q1" H 4715 3395 45  0000 L CNN
 F 1 "MOSFET-NCH-2N7002PW" H 4715 3311 45  0000 L CNN
 F 2 "SOT323" H 4550 3600 20  0001 C CNN
@@
 	4650 3000 4650 3100
 $Comp
-L power:-12V SOLC
+L power:-12V #SOLC0101
 U 1 1 5BEAB449
 P 4650 4600
-F 0 "SOLC" H 4592 4591 50  0000 R CNN
+F 0 "#SOLC0101" H 4592 4591 50  0000 R CNN
 F 1 "-12V" H 4592 4682 50  0000 R CNN
 F 2 "" H 4650 4600 50  0001 C CNN
@@
 $EndComp
 $Comp
-L power:+12V #PWR?
+L power:+12V #PWR0114
 U 1 1 5BEAB450
 P 4650 4000
-F 0 "#PWR?" H 4650 3850 50  0001 C CNN
+F 0 "#PWR0114" H 4650 3850 50  0001 C CNN
 F 1 "+12V" H 4665 4173 50  0000 C CNN
 F 2 "" H 4650 4000 50  0001 C CNN
@@
 $EndComp
 $Comp
-L SparkFun-DiscreteSemi:MOSFET-NCH-2N7002PW Q?
+L SparkFun-DiscreteSemi:MOSFET-NCH-2N7002PW Q2
 U 1 1 5BEAB457
 P 4550 4300
-F 0 "Q?" H 4715 4395 45  0000 L CNN
+F 0 "Q2" H 4715 4395 45  0000 L CNN
 F 1 "MOSFET-NCH-2N7002PW" H 4715 4311 45  0000 L CNN
 F 2 "SOT323" H 4550 4600 20  0001 C CNN
@@
 	4650 4000 4650 4100
 $Comp
-L Device:Buzzer BZ?
+L Device:Buzzer BZ1
 U 1 1 5BEADE3C
 P 4750 5700
-F 0 "BZ?" H 4903 5729 50  0000 L CNN
+F 0 "BZ1" H 4903 5729 50  0000 L CNN
 F 1 "Buzzer" H 4903 5638 50  0000 L CNN
 F 2 "" V 4725 5800 50  0001 C CNN
@@
 $EndComp
 $Comp
-L SparkFun-DiscreteSemi:MOSFET-NCH-2N7002PW Q?
+L SparkFun-DiscreteSemi:MOSFET-NCH-2N7002PW Q3
 U 1 1 5BEB292C
 P 4550 5250
-F 0 "Q?" H 4715 5345 45  0000 L CNN
+F 0 "Q3" H 4715 5345 45  0000 L CNN
 F 1 "MOSFET-NCH-2N7002PW" H 4715 5261 45  0000 L CNN
 F 2 "SOT323" H 4550 5550 20  0001 C CNN
@@
 	4350 5350 3950 5350
 $Comp
-L power:+6V #PWR?
+L power:+6V #PWR0115
 U 1 1 5BEB715A
 P 4650 4950
-F 0 "#PWR?" H 4650 4800 50  0001 C CNN
+F 0 "#PWR0115" H 4650 4800 50  0001 C CNN
 F 1 "+6V" H 4665 5123 50  0000 C CNN
 F 2 "" H 4650 4950 50  0001 C CNN
@@
 	4650 5450 4650 5600
 $Comp
-L power:GND #PWR?
+L power:GND #PWR0116
 U 1 1 5BEBE024
 P 4650 5950
-F 0 "#PWR?" H 4650 5700 50  0001 C CNN
+F 0 "#PWR0116" H 4650 5700 50  0001 C CNN
 F 1 "GND" H 4655 5777 50  0000 C CNN
 F 2 "" H 4650 5950 50  0001 C CNN
@@
 	4650 5050 4650 4950
 $Comp
-L Device:LED D?
+L Device:LED D1
 U 1 1 5BEC62B7
 P 4350 6500
-F 0 "D?" H 4341 6716 50  0000 C CNN
+F 0 "D1" H 4341 6716 50  0000 C CNN
 F 1 "LED" H 4341 6625 50  0000 C CNN
 F 2 "" H 4350 6500 50  0001 C CNN
@@
 FIX_LED
 $Comp
-L power:GND #PWR?
+L power:GND #PWR0117
 U 1 1 5BEC8E4F
 P 4050 6600
-F 0 "#PWR?" H 4050 6350 50  0001 C CNN
+F 0 "#PWR0117" H 4050 6350 50  0001 C CNN
 F 1 "GND" H 4055 6427 50  0000 C CNN
 F 2 "" H 4050 6600 50  0001 C CNN
@@
 	4500 6500 4600 6500
 $Comp
-L Device:LED D?
+L Device:LED D2
 U 1 1 5BECDE5B
 P 5750 6150
-F 0 "D?" H 5741 6366 50  0000 C CNN
+F 0 "D2" H 5741 6366 50  0000 C CNN
 F 1 "SOLP_LED" H 5741 6275 50  0000 C CNN
 F 2 "" H 5750 6150 50  0001 C CNN
@@
 A2
 $Comp
-L power:GND #PWR?
+L power:GND #PWR0118
 U 1 1 5BECDE63
 P 5450 6250
-F 0 "#PWR?" H 5450 6000 50  0001 C CNN
+F 0 "#PWR0118" H 5450 6000 50  0001 C CNN
 F 1 "GND" H 5455 6077 50  0000 C CNN
 F 2 "" H 5450 6250 50  0001 C CNN
@@
 	5900 6150 6000 6150
 $Comp
-L Device:LED D?
+L Device:LED D3
 U 1 1 5BED08A1
 P 5750 6550
-F 0 "D?" H 5741 6766 50  0000 C CNN
+F 0 "D3" H 5741 6766 50  0000 C CNN
 F 1 "SOLC_LED" H 5741 6675 50  0000 C CNN
 F 2 "" H 5750 6550 50  0001 C CNN
@@
 A3
 $Comp
-L power:GND #PWR?
+L power:GND #PWR0119
 U 1 1 5BED08A9
 P 5450 6650
-F 0 "#PWR?" H 5450 6400 50  0001 C CNN
+F 0 "#PWR0119" H 5450 6400 50  0001 C CNN
 F 1 "GND" H 5455 6477 50  0000 C CNN
 F 2 "" H 5450 6650 50  0001 C CNN
@@
 	5900 6550 6000 6550
 $Comp
-L Switch:SW_SPST SW?
+L Switch:SW_SPST SW1
 U 1 1 5BED49C4
 P 4350 850
-F 0 "SW?" H 4350 1085 50  0000 C CNN
+F 0 "SW1" H 4350 1085 50  0000 C CNN
 F 1 "EEPROM_BTN" H 4350 994 50  0000 C CNN
 F 2 "" H 4350 850 50  0001 C CNN
@@
 7
 $Comp
-L power:+5V #PWR?
+L power:+5V #PWR0120
 U 1 1 5BED5ECD
 P 4000 800
-F 0 "#PWR?" H 4000 650 50  0001 C CNN
+F 0 "#PWR0120" H 4000 650 50  0001 C CNN
 F 1 "+5V" H 4015 973 50  0000 C CNN
 F 2 "" H 4000 800 50  0001 C CNN
@@
 	4550 850  4750 850
 $Comp
-L Switch:SW_SPST SW?
+L Switch:SW_SPST SW2
 U 1 1 5BEDC896
 P 6100 3350
-F 0 "SW?" H 6100 3585 50  0000 C CNN
+F 0 "SW2" H 6100 3585 50  0000 C CNN
 F 1 "SOLP_SW" H 6100 3494 50  0000 C CNN
 F 2 "" H 6100 3350 50  0001 C CNN
@@
 A0
 $Comp
-L power:+5V #PWR?
+L power:+5V #PWR0121
 U 1 1 5BEDC89E
 P 5750 3300
-F 0 "#PWR?" H 5750 3150 50  0001 C CNN
+F 0 "#PWR0121" H 5750 3150 50  0001 C CNN
 F 1 "+5V" H 5765 3473 50  0000 C CNN
 F 2 "" H 5750 3300 50  0001 C CNN
@@
 	6300 3350 6500 3350
 $Comp
-L Switch:SW_SPST SW?
+L Switch:SW_SPST SW3
 U 1 1 5BEDFD43
 P 6100 4300
-F 0 "SW?" H 6100 4535 50  0000 C CNN
+F 0 "SW3" H 6100 4535 50  0000 C CNN
 F 1 "SOLC_SW" H 6100 4444 50  0000 C CNN
 F 2 "" H 6100 4300 50  0001 C CNN
@@
 A1
 $Comp
-L power:+5V #PWR?
+L power:+5V #PWR0122
 U 1 1 5BEDFD4B
 P 5750 4250
-F 0 "#PWR?" H 5750 4100 50  0001 C CNN
+F 0 "#PWR0122" H 5750 4100 50  0001 C CNN
 F 1 "+5V" H 5765 4423 50  0000 C CNN
 F 2 "" H 5750 4250 50  0001 C CNN
@@
 	6300 4300 6500 4300
 $Comp
-L Device:LED D?
+L Device:LED D4
 U 1 1 5BEE4EBE
 P 7750 5250
-F 0 "D?" H 7741 5466 50  0000 C CNN
+F 0 "D4" H 7741 5466 50  0000 C CNN
 F 1 "SOLP_LED" H 7741 5375 50  0000 C CNN
 F 2 "" H 7750 5250 50  0001 C CNN
@@
 $EndComp
 $Comp
-L power:GND #PWR?
+L power:GND #PWR0123
 U 1 1 5BEE4EC6
 P 7450 5350
-F 0 "#PWR?" H 7450 5100 50  0001 C CNN
+F 0 "#PWR0123" H 7450 5100 50  0001 C CNN
 F 1 "GND" H 7455 5177 50  0000 C CNN
 F 2 "" H 7450 5350 50  0001 C CNN
@@
 	7450 5250 7450 5350
 $Comp
-L Device:LED D?
+L Device:LED D5
 U 1 1 5BEE4ECF
 P 7750 5650
-F 0 "D?" H 7741 5866 50  0000 C CNN
+F 0 "D5" H 7741 5866 50  0000 C CNN
 F 1 "SOLC_LED" H 7741 5775 50  0000 C CNN
 F 2 "" H 7750 5650 50  0001 C CNN
@@
 $EndComp
 $Comp
-L power:GND #PWR?
+L power:GND #PWR0124
 U 1 1 5BEE4ED7
 P 7450 5750
-F 0 "#PWR?" H 7450 5500 50  0001 C CNN
+F 0 "#PWR0124" H 7450 5500 50  0001 C CNN
 F 1 "GND" H 7455 5577 50  0000 C CNN
 F 2 "" H 7450 5750 50  0001 C CNN
@@
 	7450 5650 7450 5750
 $Comp
-L Device:LED D?
+L Device:LED D7
 U 1 1 5BEE8A04
 P 8500 5650
-F 0 "D?" H 8491 5866 50  0000 C CNN
+F 0 "D7" H 8491 5866 50  0000 C CNN
 F 1 "SOLP_LED" H 8491 5775 50  0000 C CNN
 F 2 "" H 8500 5650 50  0001 C CNN
@@
 $EndComp
 $Comp
-L power:GND #PWR?
+L power:GND #PWR0125
 U 1 1 5BEE8A0C
 P 8800 5750
-F 0 "#PWR?" H 8800 5500 50  0001 C CNN
+F 0 "#PWR0125" H 8800 5500 50  0001 C CNN
 F 1 "GND" H 8805 5577 50  0000 C CNN
 F 2 "" H 8800 5750 50  0001 C CNN
@@
 	8650 5650 8800 5650
 $Comp
-L Device:LED D?
+L Device:LED D6
 U 1 1 5BEE8A15
 P 8500 5250
-F 0 "D?" H 8491 5466 50  0000 C CNN
+F 0 "D6" H 8491 5466 50  0000 C CNN
 F 1 "SOLC_LED" H 8491 5375 50  0000 C CNN
 F 2 "" H 8500 5250 50  0001 C CNN
@@
 	8800 5650 8800 5750
 $Comp
-L power:GND #PWR?
+L power:GND #PWR0126
 U 1 1 5BF1D48C
 P 8800 5350
-F 0 "#PWR?" H 8800 5100 50  0001 C CNN
+F 0 "#PWR0126" H 8800 5100 50  0001 C CNN
 F 1 "GND" H 8805 5177 50  0000 C CNN
 F 2 "" H 8800 5350 50  0001 C CNN
@@
 12
 $Comp
-L SparkFun-DiscreteSemi:MOSFET-NCH-2N7002PW Q?
+L SparkFun-DiscreteSemi:MOSFET-NCH-2N7002PW Q4
 U 1 1 5BF36D0B
 P 8050 4850
-F 0 "Q?" H 8215 4945 45  0000 L CNN
+F 0 "Q4" H 8215 4945 45  0000 L CNN
 F 1 "MOSFET-NCH-2N7002PW" H 8215 4861 45  0000 L CNN
 F 2 "SOT323" H 8050 5150 20  0001 C CNN
@@
 	7850 4950 7650 4950
 $Comp
-L power:+3.3V #PWR?
+L power:+3.3V #PWR0127
 U 1 1 5BF54F36
 P 8150 4450
-F 0 "#PWR?" H 8150 4300 50  0001 C CNN
+F 0 "#PWR0127" H 8150 4300 50  0001 C CNN
 F 1 "+3.3V" H 8165 4623 50  0000 C CNN
 F 2 "" H 8150 4450 50  0001 C CNN

Commit message: Add voltage regulators, schematic pdf
Parts:
- added BT1: 7.4V, symbol Device:Battery
- added C1, C2: 0.33 uF, symbol Device:C
- added C3, C4: 0.1uF, symbol Device:C
- added U5, U6: L7805, symbol Regulator_Linear:L7805
- added U7: U3V12F12, symbol RAPTOR-rescue:U3V12F12
Connections:
- net labels added: +7.5V
- wire segments 117 -> 140
Other:
- moved on the sheet: D4, D5, D6, D7

Commit message: Voltage Reg Footprints
Created the voltage regulator footprint for he 12v reg
Parts:
- Q1, Q2, Q3, Q4: symbol SparkFun-DiscreteSemi:MOSFET-NCH-2N7002PW -> RAPTOR-rescue:MOSFET-NCH-2N7002PW-SparkFun-DiscreteSemi
- U7: footprint (none) -> RAPTOR_footprints:U3V12F12
Changed lines of the file:
@@
 $EndComp
 $Comp
-L SparkFun-DiscreteSemi:MOSFET-NCH-2N7002PW Q1
+L RAPTOR-rescue:MOSFET-NCH-2N7002PW-SparkFun-DiscreteSemi Q1
 U 1 1 5BE8A581
 P 4550 3300
@@
 $EndComp
 $Comp
-L SparkFun-DiscreteSemi:MOSFET-NCH-2N7002PW Q2
+L RAPTOR-rescue:MOSFET-NCH-2N7002PW-SparkFun-DiscreteSemi Q2
 U 1 1 5BEAB457
 P 4550 4300
@@
 $EndComp
 $Comp
-L SparkFun-DiscreteSemi:MOSFET-NCH-2N7002PW Q3
+L RAPTOR-rescue:MOSFET-NCH-2N7002PW-SparkFun-DiscreteSemi Q3
 U 1 1 5BEB292C
 P 4550 5250
@@
 12
 $Comp
-L SparkFun-DiscreteSemi:MOSFET-NCH-2N7002PW Q4
+L RAPTOR-rescue:MOSFET-NCH-2N7002PW-SparkFun-DiscreteSemi Q4
 U 1 1 5BF36D0B
 P 6900 5000
@@
 F 0 "U7" H 8100 4342 50  0000 C CNN
 F 1 "U3V12F12" H 8100 4251 50  0000 C CNN
-F 2 "" H 8100 4350 50  0001 C CNN
+F 2 "RAPTOR_footprints:U3V12F12" H 8100 4350 50  0001 C CNN
 F 3 "" H 8100 4350 50  0001 C CNN
 	1    8100 4100

Commit message: Auto stash before merge of "hardware" and "origin/hardware"
Parts:
- U1: value BMP280 -> BMP280 Breakout
- U2: value BNO055 -> BNO055 Breakout
- U7: footprint RAPTOR_footprints:U3V12F12 -> (none)
Connections:
- net +5V: now also M2.2 (+)
- net +6V: no longer M2.2 (+)
- net +7.5V: now also BT1.1 (+)
- net GND: now also BT1.2 (-)
Other:
- moved on the sheet: C1, C3, D4, D5, D6, D7, M1, M2, Q4, SW1, U5, U7
