File: hardware/RAPTOR/RAPTOR.sch (KiCad schematic (older format))
At the start: 49 parts, among them J1 SOLC_CONN, J2 SOLP_CONN, J3 JST_2MM_MALE, J4 CONN_LED_FIX, J5 CONN_SOLP_LED, J6 CONN_SOLC_LED, P1 Power, P2 Analog, P3 Digital, P4 Digital, P5 CONN_01X01, P6 CONN_01X01, P7 CONN_01X01, P8 CONN_01X01, Q1 MOSFET-NCH-2N7002PW, Q2 MOSFET-NCH-2N7002PW, Q3 MOSFET-NCH-2N7002PW, Q4 MOSFET-NCH-2N7002PW, SW1 EEPROM_BTN, SW2 SOLC_SW, SW3 SOLP_SW, U1 BMP280 Breakout, U2 BNO055 Breakout, U3 OpenLog, U4 AdafruitGPS, U5 U3V12F12, U6 L4940V5

Commit message: added connectors for exterior LEDs in place of diodes
Parts:
- removed D4, D7: SOLP_LED, symbol Device:LED
- removed D5, D6: SOLC_LED, symbol Device:LED
- added J?: EXT_LED3, 1X02, symbol RAPTOR-rescue:CONN_02-SparkFun-Connectors
- added J?: EXT_LED2, 1X02, symbol RAPTOR-rescue:CONN_02-SparkFun-Connectors
- added J?: EXT_LED1, 1X02, symbol RAPTOR-rescue:CONN_02-SparkFun-Connectors
- added J?: EXT_LED0, 1X02, symbol RAPTOR-rescue:CONN_02-SparkFun-Connectors
Connections:
- wire segments 169 -> 177
Other:
- moved on the sheet: BZ1, Q3, Q4
Changed lines of the file:
@@
 L Device:Buzzer BZ1
 U 1 1 5BEADE3C
-P 3700 4600
-F 0 "BZ1" H 3853 4629 50  0000 L CNN
-F 1 "Buzzer" H 3853 4538 50  0000 L CNN
-F 2 "" V 3675 4700 50  0001 C CNN
-F 3 "~" V 3675 4700 50  0001 C CNN
-	1    3700 4600
+P 3600 5300
+F 0 "BZ1" H 3753 5329 50  0000 L CNN
+F 1 "Buzzer" H 3753 5238 50  0000 L CNN
+F 2 "" V 3575 5400 50  0001 C CNN
+F 3 "~" V 3575 5400 50  0001 C CNN
+	1    3600 5300
 	1    0    0    -1
 $EndComp
@@
 L RAPTOR-rescue:MOSFET-NCH-2N7002PW-SparkFun-DiscreteSemi Q3
 U 1 1 5BEB292C
-P 3500 5050
-F 0 "Q3" H 3665 5145 45  0000 L CNN
-F 1 "MOSFET-NCH-2N7002PW" H 3665 5061 45  0000 L CNN
-F 2 "SOT323" H 3500 5350 20  0001 C CNN
-F 3 "https://www.diodes.com/assets/Datasheets/ds11303.pdf" H 3500 5050 50  0001 C CNN
-F 4 "TRANS-11151" H 3665 4966 60  0000 L CNN "Field4"
-	1    3500 5050
-	1    0    0    -1
-$EndComp
-Text Label 2900 5150 0    50   ~ 0
+P 3400 5750
+F 0 "Q3" H 3565 5845 45  0000 L CNN
+F 1 "MOSFET-NCH-2N7002PW" H 3565 5761 45  0000 L CNN
+F 2 "SOT323" H 3400 6050 20  0001 C CNN
+F 3 "https://www.diodes.com/assets/Datasheets/ds11303.pdf" H 3400 5750 50  0001 C CNN
+F 4 "TRANS-11151" H 3565 5666 60  0000 L CNN "Field4"
+	1    3400 5750
+	1    0    0    -1
+$EndComp
+Text Label 2800 5850 0    50   ~ 0
 BZZ_DTA
 Wire Wire Line
-	3300 5150 2900 5150
-Wire Wire Line
-	3600 4700 3600 4850
+	3200 5850 2800 5850
+Wire Wire Line
+	3500 5400 3500 5550
 $Comp
 L power:GND #PWR0116
 U 1 1 5BEBE024
-P 3600 5400
-F 0 "#PWR0116" H 3600 5150 50  0001 C CNN
-F 1 "GND" H 3605 5227 50  0000 C CNN
-F 2 "" H 3600 5400 50  0001 C CNN
-F 3 "" H 3600 5400 50  0001 C CNN
-	1    3600 5400
-	1    0    0    -1
-$EndComp
-Wire Wire Line
-	3600 5250 3600 5400
-Wire Wire Line
-	3600 4500 3600 4400
+P 3500 6100
+F 0 "#PWR0116" H 3500 5850 50  0001 C CNN
+F 1 "GND" H 3505 5927 50  0000 C CNN
+F 2 "" H 3500 6100 50  0001 C CNN
+F 3 "" H 3500 6100 50  0001 C CNN
+	1    3500 6100
+	1    0    0    -1
+$EndComp
+Wire Wire Line
+	3500 5950 3500 6100
+Wire Wire Line
+	3500 5200 3500 5100
 Text Label 6450 5200 0    50   ~ 0
 FIX_LED
@@
 	4600 5200 4600 5300
 $Comp
-L Device:LED D4
-U 1 1 5BEE4EBE
-P 1050 6250
-F 0 "D4" H 1041 6466 50  0000 C CNN
-F 1 "SOLP_LED" H 1041 6375 50  0000 C CNN
-F 2 "" H 1050 6250 50  0001 C CNN
-F 3 "~" H 1050 6250 50  0001 C CNN
-	1    1050 6250
-	0    -1   -1   0
-$EndComp
-$Comp
 L power:GND #PWR0123
 U 1 1 5BEE4EC6
-P 1600 7100
-F 0 "#PWR0123" H 1600 6850 50  0001 C CNN
-F 1 "GND" H 1605 6927 50  0000 C CNN
-F 2 "" H 1600 7100 50  0001 C CNN
-F 3 "" H 1600 7100 50  0001 C CNN
-	1    1600 7100
-	1    0    0    -1
-$EndComp
-$Comp
-L Device:LED D5
-U 1 1 5BEE4ECF
-P 1400 6250
-F 0 "D5" H 1391 6466 50  0000 C CNN
-F 1 "SOLC_LED" H 1391 6375 50  0000 C CNN
-F 2 "" H 1400 6250 50  0001 C CNN
-F 3 "~" H 1400 6250 50  0001 C CNN
-	1    1400 6250
-	0    -1   -1   0
-$EndComp
-$Comp
-L Device:LED D7
-U 1 1 5BEE8A04
-P 2100 6250
-F 0 "D7" H 2091 6466 50  0000 C CNN
-F 1 "SOLP_LED" H 2091 6375 50  0000 C CNN
-F 2 "" H 2100 6250 50  0001 C CNN
-F 3 "~" H 2100 6250 50  0001 C CNN
-	1    2100 6250
-	0    -1   -1   0
-$EndComp
-$Comp
-L Device:LED D6
-U 1 1 5BEE8A15
-P 1750 6250
-F 0 "D6" H 1741 6466 50  0000 C CNN
-F 1 "SOLC_LED" H 1741 6375 50  0000 C CNN
-F 2 "" H 1750 6250 50  0001 C CNN
-F 3 "~" H 1750 6250 50  0001 C CNN
-	1    1750 6250
-	0    -1   -1   0
-$EndComp
-Text Label 1250 6950 2    50   ~ 0
+P 1600 7400
+F 0 "#PWR0123" H 1600 7150 50  0001 C CNN
+F 1 "GND" H 1605 7227 50  0000 C CNN
+F 2 "" H 1600 7400 50  0001 C CNN
+F 3 "" H 1600 7400 50  0001 C CNN
+	1    1600 7400
+	1    0    0    -1
+$EndComp
+Text Label 1250 7100 2    50   ~ 0
 LEDS_DTA
 $Comp
 L RAPTOR-rescue:MOSFET-NCH-2N7002PW-SparkFun-DiscreteSemi Q4
 U 1 1 5BF36D0B
-P 1500 6850
-F 0 "Q4" H 1665 6945 45  0000 L CNN
-F 1 "MOSFET-NCH-2N7002PW" H 1665 6861 45  0000 L CNN
-F 2 "SOT323" H 1500 7150 20  0001 C CNN
-F 3 "https://www.diodes.com/assets/Datasheets/ds11303.pdf" H 1500 6850 50  0001 C CNN
-F 4 "TRANS-11151" H 1665 6766 60  0000 L CNN "Field4"
-	1    1500 6850
+P 1500 7000
+F 0 "Q4" H 1665 7095 45  0000 L CNN
+F 1 "MOSFET-NCH-2N7002PW" H 1665 7011 45  0000 L CNN
+F 2 "SOT323" H 1500 7300 20  0001 C CNN
+F 3 "https://www.diodes.com/assets/Datasheets/ds11303.pdf" H 1500 7000 50  0001 C CNN
+F 4 "TRANS-11151" H 1665 6916 60  0000 L CNN "Field4"
+	1    1500 7000
 	1    0    0    -1
 $EndComp
@@
 F 2 "1X02" H 5050 2600 20  0001 C CNN
 F 3 "" H 5050 2350 50  0001 C CNN
-F 4 "XXX-00000" H 4822 2484 60  0000 R CNN "Field4"
+F 4 "XXX-00000" H 4822 2484 60  0001 R CNN "Field4"
 	1    5050 2350
 	-1   0    0    1
@@
 F 2 "1X02" H 5050 4050 20  0001 C CNN
 F 3 "" H 5050 3800 50  0001 C CNN
-F 4 "XXX-00000" H 4822 3934 60  0000 R CNN "Field4"
+F 4 "XXX-00000" H 4822 3934 60  0001 R CNN "Field4"
 	1    5050 3800
 	-1   0    0    1
@@
 L power:+5V #PWR017
 U 1 1 5C3D9668
-P 3600 4400
-F 0 "#PWR017" H 3600 4250 50  0001 C CNN
-F 1 "+5V" H 3615 4573 50  0000 C CNN
-F 2 "" H 3600 4400 50  0001 C CNN
-F 3 "" H 3600 4400 50  0001 C CNN
-	1    3600 4400
+P 3500 5100
+F 0 "#PWR017" H 3500 4950 50  0001 C CNN
+F 1 "+5V" H 3515 5273 50  0000 C CNN
+F 2 "" H 3500 5100 50  0001 C CNN
+F 3 "" H 3500 5100 50  0001 C CNN
+	1    3500 5100
 	1    0    0    -1
 $EndComp
@@
 F 2 "1X02" H 4950 5350 20  0001 C CNN
 F 3 "" H 4950 5100 50  0001 C CNN
-F 4 "XXX-00000" V 4990 5278 60  0000 L CNN "Field4"
+F 4 "XXX-00000" V 4990 5278 60  0001 L CNN "Field4"
 	1    4950 5100
 	0    1    1    0
@@
 F 2 "1X02" H 4950 6100 20  0001 C CNN
 F 3 "" H 4950 5850 50  0001 C CNN
-F 4 "XXX-00000" V 4990 6028 60  0000 L CNN "Field4"
+F 4 "XXX-00000" V 4990 6028 60  0001 L CNN "Field4"
 	1    4950 5850
 	0    1    1    0
@@
 F 2 "1X02" H 4950 6800 20  0001 C CNN
 F 3 "" H 4950 6550 50  0001 C CNN
-F 4 "XXX-00000" V 4990 6728 60  0000 L CNN "Field4"
+F 4 "XXX-00000" V 4990 6728 60  0001 L CNN "Field4"
 	1    4950 6550
 	0    1    1    0
@@
 F 2 "1X03" H 5150 2150 20  0001 C CNN
 F 3 "" H 5150 1750 50  0001 C CNN
-F 4 "XXX-00000" H 5106 2081 60  0000 C CNN "Field4"
+F 4 "XXX-00000" H 5106 2081 60  0001 C CNN "Field4"
 	1    5150 1750
 	1    0    0    -1
@@
 F 2 "1X03" H 5150 1500 20  0001 C CNN
 F 3 "" H 5150 1100 50  0001 C CNN
-F 4 "XXX-00000" H 5106 1431 60  0000 C CNN "Field4"
+F 4 "XXX-00000" H 5106 1431 60  0001 C CNN "Field4"
 	1    5150 1100
 	1    0    0    -1
@@
 Connection ~ 4950 3650
 Wire Wire Line
-	1600 7100 1600 7050
-Wire Wire Line
-	1600 6650 1600 6550
-Wire Wire Line
-	1600 6550 1750 6550
-Wire Wire Line
 	2100 6550 2100 6400
-Wire Wire Line
-	1750 6400 1750 6550
 Connection ~ 1750 6550
 Wire Wire Line
 	1750 6550 2100 6550
-Wire Wire Line
-	1600 6550 1400 6550
-Wire Wire Line
-	1400 6550 1400 6400
-Connection ~ 1600 6550
 Wire Wire Line
 	1050 6400 1050 6550
@@
 Wire Wire Line
 	1600 5950 1600 5900
-Wire Wire Line
-	1400 6100 1400 5950
 Connection ~ 1400 5950
 Wire Wire Line
 	1400 5950 1600 5950
-Wire Wire Line
-	1750 6100 1750 5950
 Wire Wire Line
 	1750 5950 1600 5950
@@
 Connection ~ 1750 5950
 Wire Wire Line
-	1300 6950 1150 6950
+	1300 7100 1150 7100
 $Comp
 L Regulator_Linear:L7805 U6
@@
 F 2 "1X02" H 7350 2950 20  0001 C CNN
 F 3 "" H 7350 2700 50  0001 C CNN
-F 4 "XXX-00000" H 7122 2834 60  0000 R CNN "Field4"
+F 4 "XXX-00000" H 7122 2834 60  0001 R CNN "Field4"
 	1    7350 2700
 	-1   0    0    1
@@
 Wire Wire Line
 	3800 3200 3950 3200
+$Comp
+L RAPTOR-rescue:CONN_02-SparkFun-Connectors J?
+U 1 1 5C53EBAE
+P 2250 6200
+F 0 "J?" V 2111 6378 45  0000 L CNN
+F 1 "EXT_LED3" V 2195 6378 45  0000 L CNN
+F 2 "1X02" H 2250 6450 20  0001 C CNN
+F 3 "" H 2250 6200 50  0001 C CNN
+F 4 "XXX-00000" V 2290 6378 60  0001 L CNN "Field4"
+	1    2250 6200
+	-1   0    0    1
+$EndComp
+$Comp
+L RAPTOR-rescue:CONN_02-SparkFun-Connectors J?
+U 1 1 5C54F806
+P 1850 6200
+F 0 "J?" V 1711 6378 45  0000 L CNN
+F 1 "EXT_LED2" V 1795 6378 45  0000 L CNN
+F 2 "1X02" H 1850 6450 20  0001 C CNN
+F 3 "" H 1850 6200 50  0001 C CNN
+F 4 "XXX-00000" V 1890 6378 60  0001 L CNN "Field4"
+	1    1850 6200
+	-1   0    0    1
+$EndComp
+$Comp
+L RAPTOR-rescue:CONN_02-SparkFun-Connectors J?
+U 1 1 5C557DC0
+P 1300 6300
+F 0 "J?" V 1161 6478 45  0000 L CNN
+F 1 "EXT_LED1" V 1245 6478 45  0000 L CNN
+F 2 "1X02" H 1300 6550 20  0001 C CNN
+F 3 "" H 1300 6300 50  0001 C CNN
+F 4 "XXX-00000" V 1340 6478 60  0001 L CNN "Field4"
+	1    1300 6300
+	1    0    0    -1
+$EndComp
+$Comp
+L RAPTOR-rescue:CONN_02-SparkFun-Connectors J?
+U 1 1 5C5688B4
+P 900 6300
+F 0 "J?" V 761 6478 45  0000 L CNN
+F 1 "EXT_LED0" V 845 6478 45  0000 L CNN
+F 2 "1X02" H 900 6550 20  0001 C CNN
+F 3 "" H 900 6300 50  0001 C CNN
+F 4 "XXX-00000" V 940 6478 60  0001 L CNN "Field4"
+	1    900  6300
+	1    0    0    -1
+$EndComp
+Wire Wire Line
+	2100 6100 2150 6100
+Wire Wire Line
+	2150 6100 2150 6200
+Wire Wire Line
+	2100 6400 2150 6400
+Wire Wire Line
+	2150 6400 2150 6300
+Wire Wire Line
+	1050 6100 1000 6100
+Wire Wire Line
+	1000 6100 1000 6200
+Wire Wire Line
+	1050 6400 1000 6400
+Wire Wire Line
+	1000 6400 1000 6300
+Wire Wire Line
+	1750 5950 1750 6200
+Wire Wire Line
+	1400 5950 1400 6200
+Wire Wire Line
+	1400 6300 1400 6550
+Wire Wire Line
+	1750 6300 1750 6550
+Wire Wire Line
+	1400 6550 1600 6550
+Wire Wire Line
+	1600 6550 1600 6800
+Connection ~ 1600 6550
+Wire Wire Line
+	1600 6550 1750 6550
+Wire Wire Line
+	1600 7200 1600 7400
 $EndSCHEMATC

Commit message: change to D24V550F5
Parts:
- U6: value L4940V5 -> D24V550F5; footprint Package_TO_SOT_THT:TO-220-3_Horizontal_TabDown -> (none)
- gave numbers to parts that had none: 14
Connections:
- no-connect marks 15 -> 16
Changed lines of the file:
@@
 	4600 6650 4950 6650
 $Comp
-L RAPTOR-rescue:CONN_03-SparkFun-Connectors J?
+L RAPTOR-rescue:CONN_03-SparkFun-Connectors J12
 U 1 1 5C6A99EC
 P 5150 1750
-F 0 "J?" H 5106 2260 45  0000 C CNN
+F 0 "J12" H 5106 2260 45  0000 C CNN
 F 1 "SRVOR_CONN" H 5106 2176 45  0000 C CNN
 F 2 "1X03" H 5150 2150 20  0001 C CNN
@@
 $EndComp
 $Comp
-L RAPTOR-rescue:CONN_03-SparkFun-Connectors J?
+L RAPTOR-rescue:CONN_03-SparkFun-Connectors J11
 U 1 1 5C6B1587
 P 5150 1100
-F 0 "J?" H 5106 1610 45  0000 C CNN
+F 0 "J11" H 5106 1610 45  0000 C CNN
 F 1 "SRVOL_CONN" H 5106 1526 45  0000 C CNN
 F 2 "1X03" H 5150 1500 20  0001 C CNN
@@
 P 3550 850
 F 0 "U6" H 3550 1092 50  0000 C CNN
-F 1 "L4940V5" H 3550 1001 50  0000 C CNN
-F 2 "Package_TO_SOT_THT:TO-220-3_Horizontal_TabDown" H 3575 700 50  0001 L CIN
+F 1 "D24V550F5" H 3550 1001 50  0000 C CNN
+F 2 "" H 3575 700 50  0001 L CIN
 F 3 "http://www.st.com/content/ccc/resource/technical/document/datasheet/41/4f/b3/b0/12/d4/47/88/CD00000444.pdf/files/CD00000444.pdf/jcr:content/translations/en.CD00000444.pdf" H 3550 800 50  0001 C CNN
 	1    3550 850
@@
 $EndComp
 $Comp
-L RAPTOR-rescue:100OHM-0603-1_10W-1%-SparkFun-Resistors R?
+L RAPTOR-rescue:100OHM-0603-1_10W-1%-SparkFun-Resistors R4
 U 1 1 5C409EAA
 P 6000 6650
-F 0 "R?" H 6000 6950 45  0000 C CNN
+F 0 "R4" H 6000 6950 45  0000 C CNN
 F 1 "100OHM-0603-1_10W-1%" H 6000 6866 45  0000 C CNN
 F 2 "0603" H 6000 6800 20  0001 C CNN
@@
 $EndComp
 $Comp
-L RAPTOR-rescue:100OHM-0603-1_10W-1%-SparkFun-Resistors R?
+L RAPTOR-rescue:100OHM-0603-1_10W-1%-SparkFun-Resistors R3
 U 1 1 5C409F6D
 P 6000 5950
-F 0 "R?" H 6000 6250 45  0000 C CNN
+F 0 "R3" H 6000 6250 45  0000 C CNN
 F 1 "100OHM-0603-1_10W-1%" H 6000 6166 45  0000 C CNN
 F 2 "0603" H 6000 6100 20  0001 C CNN
@@
 $EndComp
 $Comp
-L RAPTOR-rescue:100OHM-0603-1_10W-1%-SparkFun-Resistors R?
+L RAPTOR-rescue:100OHM-0603-1_10W-1%-SparkFun-Resistors R2
 U 1 1 5C411D44
 P 6000 5200
-F 0 "R?" H 6000 5500 45  0000 C CNN
+F 0 "R2" H 6000 5500 45  0000 C CNN
 F 1 "100OHM-0603-1_10W-1%" H 6000 5416 45  0000 C CNN
 F 2 "0603" H 6000 5350 20  0001 C CNN
@@
 $EndComp
 $Comp
-L RAPTOR-rescue:20OHM-0603-1_10W-1%-SparkFun-Resistors R?
+L RAPTOR-rescue:20OHM-0603-1_10W-1%-SparkFun-Resistors R1
 U 1 1 5C41AD57
 P 1600 5700
-F 0 "R?" V 1505 5768 45  0000 L CNN
+F 0 "R1" V 1505 5768 45  0000 L CNN
 F 1 "20OHM-0603-1_10W-1%" V 1589 5768 45  0000 L CNN
 F 2 "0603" H 1600 5850 20  0001 C CNN
@@
 $EndComp
 $Comp
-L RAPTOR-rescue:MOSFET-NCH-2N7002PW-SparkFun-DiscreteSemi Q?
+L RAPTOR-rescue:MOSFET-NCH-2N7002PW-SparkFun-DiscreteSemi Q5
 U 1 1 5C45C6C5
 P 7150 3150
-F 0 "Q?" H 7315 3245 45  0000 L CNN
+F 0 "Q5" H 7315 3245 45  0000 L CNN
 F 1 "MOSFET-NCH-2N7002PW" H 7315 3161 45  0000 L CNN
 F 2 "SOT323" H 7150 3450 20  0001 C CNN
@@
 	6950 3250 6650 3250
 $Comp
-L power:GND #PWR?
+L power:GND #PWR028
 U 1 1 5C45C6CF
 P 7250 3850
-F 0 "#PWR?" H 7250 3600 50  0001 C CNN
+F 0 "#PWR028" H 7250 3600 50  0001 C CNN
 F 1 "GND" H 7255 3677 50  0000 C CNN
 F 2 "" H 7250 3850 50  0001 C CNN
@@
 $EndComp
 $Comp
-L RAPTOR-rescue:CONN_02-SparkFun-Connectors J?
+L RAPTOR-rescue:CONN_02-SparkFun-Connectors J13
 U 1 1 5C45C6DE
 P 7350 2700
-F 0 "J?" H 7122 2655 45  0000 R CNN
+F 0 "J13" H 7122 2655 45  0000 R CNN
 F 1 "HOTWIRE_CONN" H 7122 2739 45  0000 R CNN
 F 2 "1X02" H 7350 2950 20  0001 C CNN
@@
 HOTWIRE
 $Comp
-L RAPTOR-rescue:4.7KOHM-0603-1_10W-1%-SparkFun-Resistors R?
+L RAPTOR-rescue:4.7KOHM-0603-1_10W-1%-SparkFun-Resistors R8
 U 1 1 5C476CBF
 P 7250 3600
-F 0 "R?" V 7155 3668 45  0000 L CNN
+F 0 "R8" V 7155 3668 45  0000 L CNN
 F 1 "4.7KOHM-0603-1_10W-1%" V 7239 3668 45  0000 L CNN
 F 2 "0603" H 7250 3750 20  0001 C CNN
@@
 	7250 2450 7250 2700
 $Comp
-L power:+7.5V #PWR?
+L power:+7.5V #PWR027
 U 1 1 5C4B44D8
 P 7250 2450
-F 0 "#PWR?" H 7250 2300 50  0001 C CNN
+F 0 "#PWR027" H 7250 2300 50  0001 C CNN
 F 1 "+7.5V" H 7265 2623 50  0001 C CNN
 F 2 "" H 7250 2450 50  0001 C CNN
@@
 $EndComp
 $Comp
-L Switch:SW_SPST SW?
+L Switch:SW_SPST SW4
 U 1 1 5C4BDD6E
 P 3600 3200
-F 0 "SW?" H 3600 3435 50  0000 C CNN
+F 0 "SW4" H 3600 3435 50  0000 C CNN
 F 1 "RBF" H 3600 3344 50  0000 C CNN
 F 2 "" H 3600 3200 50  0001 C CNN
@@
 	3800 3200 3950 3200
 $Comp
-L RAPTOR-rescue:CONN_02-SparkFun-Connectors J?
+L RAPTOR-rescue:CONN_02-SparkFun-Connectors J10
 U 1 1 5C53EBAE
 P 2250 6200
-F 0 "J?" V 2111 6378 45  0000 L CNN
+F 0 "J10" V 2111 6378 45  0000 L CNN
 F 1 "EXT_LED3" V 2195 6378 45  0000 L CNN
 F 2 "1X02" H 2250 6450 20  0001 C CNN
@@
 $EndComp
 $Comp
-L RAPTOR-rescue:CONN_02-SparkFun-Connectors J?
+L RAPTOR-rescue:CONN_02-SparkFun-Connectors J9
 U 1 1 5C54F806
 P 1850 6200
-F 0 "J?" V 1711 6378 45  0000 L CNN
+F 0 "J9" V 1711 6378 45  0000 L CNN
 F 1 "EXT_LED2" V 1795 6378 45  0000 L CNN
 F 2 "1X02" H 1850 6450 20  0001 C CNN
@@
 $EndComp
 $Comp
-L RAPTOR-rescue:CONN_02-SparkFun-Connectors J?
+L RAPTOR-rescue:CONN_02-SparkFun-Connectors J8
 U 1 1 5C557DC0
 P 1300 6300
-F 0 "J?" V 1161 6478 45  0000 L CNN
+F 0 "J8" V 1161 6478 45  0000 L CNN
 F 1 "EXT_LED1" V 1245 6478 45  0000 L CNN
 F 2 "1X02" H 1300 6550 20  0001 C CNN
@@
 $EndComp
 $Comp
-L RAPTOR-rescue:CONN_02-SparkFun-Connectors J?
+L RAPTOR-rescue:CONN_02-SparkFun-Connectors J7
 U 1 1 5C5688B4
 P 900 6300
-F 0 "J?" V 761 6478 45  0000 L CNN
+F 0 "J7" V 761 6478 45  0000 L CNN
 F 1 "EXT_LED0" V 845 6478 45  0000 L CNN
 F 2 "1X02" H 900 6550 20  0001 C CNN
@@
 Wire Wire Line
 	1600 7200 1600 7400
+NoConn ~ 1950 2450
 $EndSCHEMATC

Commit message: make everything connectors
Parts:
- removed SW1: EEPROM_BTN, symbol Switch:SW_SPST
- removed SW2: SOLC_SW, symbol Switch:SW_SPST
- removed SW3: SOLP_SW, symbol Switch:SW_SPST
- removed SW4: RBF, symbol Switch:SW_SPST
- added J?: EEPROM_BTN_CONN, 1X02, symbol RAPTOR-rescue:CONN_02-SparkFun-Connectors
- added J?: SOLC_SW_CONN, 1X03, symbol RAPTOR-rescue:CONN_03-SparkFun-Connectors
- added J?: SOLP_SW_CONN, 1X03, symbol RAPTOR-rescue:CONN_03-SparkFun-Connectors
- added J?: RBF_CONN, 1X03, symbol RAPTOR-rescue:CONN_03-SparkFun-Connectors
Connections:
- wire segments 177 -> 184
- no-connect marks 16 -> 19
Changed lines of the file:
@@
 Wire Wire Line
 	6200 5200 6450 5200
-$Comp
-L Switch:SW_SPST SW1
-U 1 1 5C539DBE
-P 8700 4050
-F 0 "SW1" H 8700 4285 50  0000 C CNN
-F 1 "EEPROM_BTN" H 8700 4194 50  0000 C CNN
-F 2 "" H 8700 4050 50  0001 C CNN
-F 3 "" H 8700 4050 50  0001 C CNN
-	1    8700 4050
-	0    1    1    0
-$EndComp
 Text Label 8350 4300 0    50   ~ 0
 EEPROM_BTN
@@
 $EndComp
 Wire Wire Line
-	8700 4250 8700 4300
-Wire Wire Line
 	8700 4750 8700 4850
-Wire Wire Line
-	8700 3850 8700 3700
 Wire Wire Line
 	8350 4300 8700 4300
@@
 Wire Wire Line
 	8700 4300 8700 4350
-$Comp
-L Switch:SW_SPST SW3
-U 1 1 5C542020
-P 9850 4050
-F 0 "SW3" H 9850 4285 50  0000 C CNN
-F 1 "SOLP_SW" H 9850 4194 50  0000 C CNN
-F 2 "" H 9850 4050 50  0001 C CNN
-F 3 "" H 9850 4050 50  0001 C CNN
-	1    9850 4050
-	0    1    1    0
-$EndComp
 Text Label 9500 4300 0    50   ~ 0
 SOLP_SW
@@
 $EndComp
 Wire Wire Line
-	9850 4250 9850 4300
-Wire Wire Line
 	9850 4750 9850 4850
-Wire Wire Line
-	9850 3850 9850 3700
 Wire Wire Line
 	9500 4300 9850 4300
@@
 Wire Wire Line
 	9850 4300 9850 4350
-$Comp
-L Switch:SW_SPST SW2
-U 1 1 5C54A1B2
-P 9250 5450
-F 0 "SW2" H 9250 5685 50  0000 C CNN
-F 1 "SOLC_SW" H 9250 5594 50  0000 C CNN
-F 2 "" H 9250 5450 50  0001 C CNN
-F 3 "" H 9250 5450 50  0001 C CNN
-	1    9250 5450
-	0    1    1    0
-$EndComp
 Text Label 8900 5700 0    50   ~ 0
 SOLC_SW
@@
 $EndComp
 Wire Wire Line
-	9250 5650 9250 5700
-Wire Wire Line
 	9250 6150 9250 6250
 Wire Wire Line
-	9250 5250 9250 5100
-Wire Wire Line
 	8900 5700 9250 5700
-Connection ~ 9250 5700
 Wire Wire Line
 	9250 5700 9250 5750
@@
 Wire Wire Line
 	4600 5950 4600 6050
-Wire Wire Line
-	6200 5950 6450 5950
 $Comp
 L RAPTOR-rescue:CONN_02-SparkFun-Connectors J5
@@
 U 1 1 5C6A99EC
 P 5150 1750
-F 0 "J12" H 5106 2260 45  0000 C CNN
-F 1 "SRVOR_CONN" H 5106 2176 45  0000 C CNN
+F 0 "J12" H 5050 2150 45  0000 C CNN
+F 1 "SRVOR_CONN" H 5050 2050 45  0000 C CNN
 F 2 "1X03" H 5150 2150 20  0001 C CNN
 F 3 "" H 5150 1750 50  0001 C CNN
@@
 U 1 1 5C6B1587
 P 5150 1100
-F 0 "J11" H 5106 1610 45  0000 C CNN
-F 1 "SRVOL_CONN" H 5106 1526 45  0000 C CNN
+F 0 "J11" H 5050 1500 45  0000 C CNN
+F 1 "SRVOL_CONN" H 5050 1400 45  0000 C CNN
 F 2 "1X03" H 5150 1500 20  0001 C CNN
 F 3 "" H 5150 1100 50  0001 C CNN
@@
 $EndComp
 $Comp
-L Switch:SW_SPST SW4
-U 1 1 5C4BDD6E
-P 3600 3200
-F 0 "SW4" H 3600 3435 50  0000 C CNN
-F 1 "RBF" H 3600 3344 50  0000 C CNN
-F 2 "" H 3600 3200 50  0001 C CNN
-F 3 "" H 3600 3200 50  0001 C CNN
-	1    3600 3200
-	1    0    0    -1
-$EndComp
-Wire Wire Line
-	3250 3200 3400 3200
-Wire Wire Line
-	3800 3200 3950 3200
-$Comp
 L RAPTOR-rescue:CONN_02-SparkFun-Connectors J10
 U 1 1 5C53EBAE
@@
 	1600 7200 1600 7400
 NoConn ~ 1950 2450
+Wire Wire Line
+	6200 5950 6450 5950
+$Comp
+L RAPTOR-rescue:CONN_02-SparkFun-Connectors J?
+U 1 1 5C767459
+P 8800 4000
+F 0 "J?" H 8572 3955 45  0000 R CNN
+F 1 "EEPROM_BTN_CONN" H 8572 4039 45  0000 R CNN
+F 2 "1X02" H 8800 4250 20  0001 C CNN
+F 3 "" H 8800 4000 50  0001 C CNN
+F 4 "XXX-00000" H 8572 4134 60  0001 R CNN "Field4"
+	1    8800 4000
+	-1   0    0    1
+$EndComp
+Wire Wire Line
+	8700 3700 8700 4000
+$Comp
+L RAPTOR-rescue:CONN_03-SparkFun-Connectors J?
+U 1 1 5C785495
+P 9450 5350
+F 0 "J?" V 9200 5450 45  0000 C CNN
+F 1 "SOLC_SW_CONN" V 9100 5450 45  0000 C CNN
+F 2 "1X03" H 9450 5750 20  0001 C CNN
+F 3 "https://omronfs.omron.com/en_US/ecb/products/pdf/en-d2fs.pdf" H 9450 5350 50  0001 C CNN
+F 4 "XXX-00000" H 9406 5681 60  0001 C CNN "Field4"
+	1    9450 5350
+	-1   0    0    1
+$EndComp
+Wire Wire Line
+	8700 4250 8700 4300
+Wire Wire Line
+	8700 4100 8700 4300
+Wire Wire Line
+	9350 5350 9250 5350
+Wire Wire Line
+	9250 5100 9250 5350
+Wire Wire Line
+	9350 5450 9250 5450
+Wire Wire Line
+	9250 5450 9250 5700
+Connection ~ 9250 5700
+NoConn ~ 9350 5550
+$Comp
+L RAPTOR-rescue:CONN_03-SparkFun-Connectors J?
+U 1 1 5C7DB3E4
+P 10050 3950
+F 0 "J?" V 9800 4050 45  0000 C CNN
+F 1 "SOLP_SW_CONN" V 9700 4050 45  0000 C CNN
+F 2 "1X03" H 10050 4350 20  0001 C CNN
+F 3 "https://omronfs.omron.com/en_US/ecb/products/pdf/en-d2fs.pdf" H 10050 3950 50  0001 C CNN
+F 4 "XXX-00000" H 10006 4281 60  0001 C CNN "Field4"
+	1    10050 3950
+	-1   0    0    1
+$EndComp
+Wire Wire Line
+	9950 3950 9850 3950
+Wire Wire Line
+	9950 4050 9850 4050
+NoConn ~ 9950 4150
+Wire Wire Line
+	9850 4050 9850 4300
+Wire Wire Line
+	9850 3700 9850 3950
+$Comp
+L RAPTOR-rescue:CONN_03-SparkFun-Connectors J?
+U 1 1 5C7F97C7
+P 3500 3050
+F 0 "J?" V 3250 3150 45  0000 C CNN
+F 1 "RBF_CONN" H 3400 3350 45  0000 C CNN
+F 2 "1X03" H 3500 3450 20  0001 C CNN
+F 3 "https://omronfs.omron.com/en_US/ecb/products/pdf/en-d2fs.pdf" H 3500 3050 50  0001 C CNN
+F 4 "XXX-00000" H 3456 3381 60  0001 C CNN "Field4"
+	1    3500 3050
+	0    1    1    0
+$EndComp
+NoConn ~ 3700 3150
+Wire Wire Line
+	3500 3150 3500 3200
+Wire Wire Line
+	3250 3200 3500 3200
+Wire Wire Line
+	3600 3150 3600 3200
+Wire Wire Line
+	3600 3200 3950 3200
 $EndSCHEMATC

Commit message: remove capacitors from circuit
Parts:
- removed C2: 0.33 uF, symbol Device:C
- removed C4: 0.1uF, symbol Device:C
- BZ1: footprint (none) -> Buzzer_Beeper:Buzzer_12x9.5RM7.6
- D8, D9: footprint DIODE-1N4148 -> Silicon-Custom:DIODE-1N4148
- J1, J10, J13, J2, J4, J5, J6, J7, J8, J9: footprint 1X02 -> Connectors:1X02
- J11, J12: footprint 1X03 -> Connectors:1X03
- J14, J16, J17: renamed from J?; footprint 1X03 -> Connectors:1X03
- J15: renamed from J?; footprint 1X02 -> Connectors:1X02
- Q1, Q2, Q3, Q4, Q5: footprint SOT323 -> Silicon-Standard:SOT323
Connections:
- wire segments 184 -> 177
Other:
- moved on the sheet: U5
