File: hardware/RAPTOR/_saved_RAPTOR.sch (KiCad schematic (older format))
At the start: 47 parts, among them J1 SOLC_CONN, J10 EXT_LED3, J11 SRVOL_CONN, J12 SRVOR_CONN, J13 HOTWIRE_CONN, J14 RBF_CONN, J15 EEPROM_BTN_CONN, J16 SOLC_SW_CONN, J17 SOLP_SW_CONN, J18 CONN_BUZZER, J2 SOLP_CONN, J3 JST_2MM_MALE, J4 CONN_LED_FIX, J5 CONN_SOLP_LED, J6 CONN_SOLC_LED, J7 EXT_LED0, J8 EXT_LED1, J9 EXT_LED2, P1 Power, P2 Analog, P3 Digital, P4 Digital, P5 CONN_01X01, P6 CONN_01X01, P7 CONN_01X01, P8 CONN_01X01, Q1 MOSFET-NCH-STQ2NK60ZR-AP, Q2 MOSFET-NCH-STQ2NK60ZR-AP, Q3 MOSFET-NCH-STQ2NK60ZR-AP, Q4 MOSFET-NCH-STQ2NK60ZR-AP, Q5 MOSFET-NCH-STQ2NK60ZR-AP, U1 BMP280 Breakout, U2 BNO055 Breakout, U3 OpenLog, U4 AdafruitGPS, U5 U3V12F12, U6 D24V550F5

Commit message: merge
Parts:
- J1, J10, J13, J14, J15, J16, J17, J18, J2, J4, J5, J6, J7, J8, J9: footprint Connectors:1X02 -> RAPTOR_footprints:Molex-2pin
- J11, J12: footprint Connectors:1X03 -> RAPTOR_footprints:Molex-MOTOR
Changed lines of the file:
@@
 F 0 "J2" H 4822 2305 45  0000 R CNN
 F 1 "SOLP_CONN" H 4822 2389 45  0000 R CNN
-F 2 "Connectors:1X02" H 5050 2600 20  0001 C CNN
+F 2 "RAPTOR_footprints:Molex-2pin" H 5050 2600 20  0001 C CNN
 F 3 "" H 5050 2350 50  0001 C CNN
 F 4 "XXX-00000" H 4822 2484 60  0001 R CNN "Field4"
@@
 F 0 "J1" H 4822 3755 45  0000 R CNN
 F 1 "SOLC_CONN" H 4822 3839 45  0000 R CNN
-F 2 "Connectors:1X02" H 5050 4050 20  0001 C CNN
+F 2 "RAPTOR_footprints:Molex-2pin" H 5050 4050 20  0001 C CNN
 F 3 "" H 5050 3800 50  0001 C CNN
 F 4 "XXX-00000" H 4822 3934 60  0001 R CNN "Field4"
@@
 F 0 "J4" V 4811 5278 45  0000 L CNN
 F 1 "CONN_LED_FIX" V 4895 5278 45  0000 L CNN
-F 2 "Connectors:1X02" H 4950 5350 20  0001 C CNN
+F 2 "RAPTOR_footprints:Molex-2pin" H 4950 5350 20  0001 C CNN
 F 3 "" H 4950 5100 50  0001 C CNN
 F 4 "XXX-00000" V 4990 5278 60  0001 L CNN "Field4"
@@
 F 0 "J5" V 4811 6028 45  0000 L CNN
 F 1 "CONN_SOLP_LED" V 4895 6028 45  0000 L CNN
-F 2 "Connectors:1X02" H 4950 6100 20  0001 C CNN
+F 2 "RAPTOR_footprints:Molex-2pin" H 4950 6100 20  0001 C CNN
 F 3 "" H 4950 5850 50  0001 C CNN
 F 4 "XXX-00000" V 4990 6028 60  0001 L CNN "Field4"
@@
 F 0 "J6" V 4811 6728 45  0000 L CNN
 F 1 "CONN_SOLC_LED" V 4895 6728 45  0000 L CNN
-F 2 "Connectors:1X02" H 4950 6800 20  0001 C CNN
+F 2 "RAPTOR_footprints:Molex-2pin" H 4950 6800 20  0001 C CNN
 F 3 "" H 4950 6550 50  0001 C CNN
 F 4 "XXX-00000" V 4990 6728 60  0001 L CNN "Field4"
@@
 F 0 "J12" H 5050 2150 45  0000 C CNN
 F 1 "SRVOR_CONN" H 5050 2050 45  0000 C CNN
-F 2 "Connectors:1X03" H 5150 2150 20  0001 C CNN
+F 2 "RAPTOR_footprints:Molex-MOTOR" H 5150 2150 20  0001 C CNN
 F 3 "" H 5150 1750 50  0001 C CNN
 F 4 "XXX-00000" H 5106 2081 60  0001 C CNN "Field4"
@@
 F 0 "J11" H 5050 1500 45  0000 C CNN
 F 1 "SRVOL_CONN" H 5050 1400 45  0000 C CNN
-F 2 "Connectors:1X03" H 5150 1500 20  0001 C CNN
+F 2 "RAPTOR_footprints:Molex-MOTOR" H 5150 1500 20  0001 C CNN
 F 3 "" H 5150 1100 50  0001 C CNN
 F 4 "XXX-00000" H 5106 1431 60  0001 C CNN "Field4"
@@
 F 0 "J13" H 7122 2655 45  0000 R CNN
 F 1 "HOTWIRE_CONN" H 7122 2739 45  0000 R CNN
-F 2 "Connectors:1X02" H 7350 2950 20  0001 C CNN
+F 2 "RAPTOR_footprints:Molex-2pin" H 7350 2950 20  0001 C CNN
 F 3 "" H 7350 2700 50  0001 C CNN
 F 4 "XXX-00000" H 7122 2834 60  0001 R CNN "Field4"
@@
 F 0 "J10" V 2111 6378 45  0000 L CNN
 F 1 "EXT_LED3" V 2195 6378 45  0000 L CNN
-F 2 "Connectors:1X02" H 2250 6450 20  0001 C CNN
+F 2 "RAPTOR_footprints:Molex-2pin" H 2250 6450 20  0001 C CNN
 F 3 "" H 2250 6200 50  0001 C CNN
 F 4 "XXX-00000" V 2290 6378 60  0001 L CNN "Field4"
@@
 F 0 "J9" V 1711 6378 45  0000 L CNN
 F 1 "EXT_LED2" V 1795 6378 45  0000 L CNN
-F 2 "Connectors:1X02" H 1850 6450 20  0001 C CNN
+F 2 "RAPTOR_footprints:Molex-2pin" H 1850 6450 20  0001 C CNN
 F 3 "" H 1850 6200 50  0001 C CNN
 F 4 "XXX-00000" V 1890 6378 60  0001 L CNN "Field4"
@@
 F 0 "J8" V 1161 6478 45  0000 L CNN
 F 1 "EXT_LED1" V 1245 6478 45  0000 L CNN
-F 2 "Connectors:1X02" H 1300 6550 20  0001 C CNN
+F 2 "RAPTOR_footprints:Molex-2pin" H 1300 6550 20  0001 C CNN
 F 3 "" H 1300 6300 50  0001 C CNN
 F 4 "XXX-00000" V 1340 6478 60  0001 L CNN "Field4"
@@
 F 0 "J7" V 761 6478 45  0000 L CNN
 F 1 "EXT_LED0" V 845 6478 45  0000 L CNN
-F 2 "Connectors:1X02" H 900 6550 20  0001 C CNN
+F 2 "RAPTOR_footprints:Molex-2pin" H 900 6550 20  0001 C CNN
 F 3 "" H 900 6300 50  0001 C CNN
 F 4 "XXX-00000" V 940 6478 60  0001 L CNN "Field4"
@@
 F 0 "J15" H 8572 3955 45  0000 R CNN
 F 1 "EEPROM_BTN_CONN" H 8572 4039 45  0000 R CNN
-F 2 "Connectors:1X02" H 8800 4250 20  0001 C CNN
+F 2 "RAPTOR_footprints:Molex-2pin" H 8800 4250 20  0001 C CNN
 F 3 "" H 8800 4000 50  0001 C CNN
 F 4 "XXX-00000" H 8572 4134 60  0001 R CNN "Field4"
@@
 F 0 "J18" V 3461 5428 45  0000 L CNN
 F 1 "CONN_BUZZER" V 3545 5428 45  0000 L CNN
-F 2 "Connectors:1X02" H 3600 5500 20  0001 C CNN
+F 2 "RAPTOR_footprints:Molex-2pin" H 3600 5500 20  0001 C CNN
 F 3 "" H 3600 5250 50  0001 C CNN
 F 4 "XXX-00000" V 3640 5428 60  0001 L CNN "Field4"
@@
 F 0 "J17" H 9822 3905 45  0000 R CNN
 F 1 "SOLP_SW_CONN" H 9822 3989 45  0000 R CNN
-F 2 "Connectors:1X02" H 10050 4200 20  0001 C CNN
+F 2 "RAPTOR_footprints:Molex-2pin" H 10050 4200 20  0001 C CNN
 F 3 "" H 10050 3950 50  0001 C CNN
 F 4 "XXX-00000" H 9822 4084 60  0001 R CNN "Field4"
@@
 F 0 "J16" H 9222 5305 45  0000 R CNN
 F 1 "SOLC_SW_CONN" H 9222 5389 45  0000 R CNN
-F 2 "Connectors:1X02" H 9450 5600 20  0001 C CNN
+F 2 "RAPTOR_footprints:Molex-2pin" H 9450 5600 20  0001 C CNN
 F 3 "" H 9450 5350 50  0001 C CNN
 F 4 "XXX-00000" H 9222 5484 60  0001 R CNN "Field4"
@@
 F 0 "J14" H 3272 3005 45  0000 R CNN
 F 1 "RBF_CONN" V 3250 3400 45  0000 R CNN
-F 2 "Connectors:1X02" H 3500 3300 20  0001 C CNN
+F 2 "RAPTOR_footprints:Molex-2pin" H 3500 3300 20  0001 C CNN
 F 3 "" H 3500 3050 50  0001 C CNN
 F 4 "XXX-00000" H 3272 3184 60  0001 R CNN "Field4"
